Commit message: Changed aux wheels

File: urdf/lmwr-diffdrive.urdf.xacro (robot description, xacro)
@@ -44,5 +44,6 @@
     <link name="${side}_aux_wheel">
       <visual>
-        <origin xyz="0 ${reflect*aux_wheel_width/2} 0" rpy="${pi/2} 0 0" />
+        <!-- origin xyz="0 ${reflect*aux_wheel_width/2} 0" rpy="${pi/2} 0 0" / -->
+        <origin xyz="0 0 0" rpy="${pi/2} 0 0" />
         <geometry>
           <cylinder radius="${aux_wheel_radius}" length="${aux_wheel_width}"/>
@@ -51,5 +52,6 @@
       </visual>
       <collision>
-        <origin xyz="0 ${reflect*aux_wheel_width/2} 0" rpy="${pi/2} 0 0" />
+        <!-- origin xyz="0 ${reflect*aux_wheel_width/2} 0" rpy="${pi/2} 0 0" / -->
+        <origin xyz="0 0 0" rpy="${pi/2} 0 0" />
         <geometry>
           <cylinder radius="${aux_wheel_radius}" length="${aux_wheel_width}"/>
@@ -62,5 +64,6 @@
       <parent link="${side}_front_support"/>
       <child link="${side}_aux_wheel"/>
-      <origin xyz="0 ${reflect*0.01} -0.06" rpy="0 0 0"/>
+      <origin xyz="-0.03 0 -0.06" rpy="0 0 0"/>
+      <!-- origin xyz="-0.03 0 -0.06" rpy="0 0 0"/ -->
     </joint>
     <!-- This block provides the simulator (Gazebo) with information on a few additional
@@ -74,5 +77,5 @@
     </gazebo>
   </xacro:macro>
-  <xacro:macro name="support" params="side reflect">
+  <xacro:macro name="support" params="side displacement reflect">
     <link name="${side}_front_support">
       <visual>
@@ -80,5 +83,5 @@
           <box size="0.05 0.01 0.08"/>
         </geometry>
-        <origin xyz="0 0 -0.04"/>
+        <origin xyz="0 ${displacement} -0.04"/>
         <material name="white"/>
       </visual>
@@ -87,5 +90,5 @@
           <box size="0.05 0.01 0.08"/>
         </geometry>
-        <origin xyz="0 0 -0.04"/>
+        <origin xyz="0 ${displacement} -0.04"/>
       </collision>
       <xacro:default_inertial mass="0.2"/>
@@ -145,6 +148,6 @@
   <xacro:traction_wheel side="left" reflect="-1"/>
   <xacro:traction_wheel side="right" reflect="1"/>
-  <xacro:support side="left" reflect="-1" />
-  <xacro:support side="right" reflect="1" />
+  <xacro:support side="left" displacement="${traction_wheel_width/2}" reflect="-1" />
+  <xacro:support side="right" displacement="${-traction_wheel_width/2}" reflect="1" />
   <!-- Gazebo plugin for ROS Control -->
   <gazebo>
