Commit message: Added inertial macros, tango urdf, refined lmwr

File: urdf/tango.urdf.xacro (robot description, xacro)
@@ -1,27 +1,43 @@
 <?xml version="1.0"?>
-<robot name="lmwr_diff_ultra_xacro" xmlns:xacro="http://ros.org/wiki/xacro">
-  <xacro:property name="body_lenght" value="0.7" />
-  <xacro:property name="body_width" value="0.4" />
-  <xacro:property name="body_height" value="0.25" />
-  <xacro:property name="traction_wheel_radius" value="0.11" />
-  <xacro:property name="traction_wheel_width" value="0.05" />
-  <xacro:property name="aux_wheel_radius" value="0.04" />
-  <xacro:property name="aux_wheel_width" value="0.03" />
-  <xacro:property name="support_lenght" value="0.6" />
-  <xacro:property name="baselen" value="0.4" />
-  <xacro:property name="wheeldiam" value="0.07" />
+<robot name="tango_xacro" xmlns:xacro="http://ros.org/wiki/xacro">
+  <xacro:property name="body_diameter" value="0.3" />
+  <xacro:property name="body_height" value="0.08" />
+  <xacro:property name="traction_wheel_radius" value="0.03" />
+  <xacro:property name="traction_wheel_width" value="0.01" />
+  <xacro:property name="aux_wheel_radius" value="0.03" />
   <xacro:property name="camera_link" value="0.05" />
   <xacro:include filename="materials.xacro" />
   <xacro:include filename="inertials.xacro" />
+  <!-- material name="blue">
+    <color rgba="0 0 0.8 1"/>
+  </material>
+  <material name="black">
+    <color rgba="0 0 0 1"/>
+  </material>
+  <material name="green">
+    <color rgba="0 1 0 1"/>
+  </material>
+  <material name="grey">
+    <color rgba=".2 .2 .2 1"/>
+  </material>
+  <material name="white">
+    <color rgba="1 1 1 1"/>
+  </material -->
+  <xacro:macro name="inertial_cube" params="mass">
+    <inertial>
+      <mass value="${mass}" />
+      <inertia ixx="1.0" ixy="0.0" ixz="0.0" iyy="1.0" iyz="0.0" izz="1.0" />
+    </inertial>
+  </xacro:macro>
   <link name="main_body">
     <visual>
       <geometry>
-        <box size="${body_lenght} ${body_width} ${body_height}"/>
-      </geometry>
-      <material name="blue"/>
+        <cylinder radius="${body_diameter/2}" length="${body_height}"/>
+      </geometry>
+      <material name="black"/>
     </visual>
     <collision>
       <geometry>
-        <box size="${body_lenght} ${body_width} ${body_height}"/>
+        <cylinder radius="${body_diameter/2}" length="${body_height}"/>
       </geometry>
     </collision>
@@ -43,36 +59,36 @@
     </collision>
     <!-- inertial>
-      <mass value="13" />
-      <inertia ixx="0.24" ixy="0.0" ixz="0.0" iyy="0.6" iyz="0.0" izz="0.7" />
+      <mass value="2" />
+      <inertia ixx="0.002" ixy="0.0" ixz="0.0" iyy="0.002" iyz="0.0" izz="0.01" />
     </inertial -->
-    <xacro:inertial_cuboid mass="13" len="${body_lenght}" width="${body_width}" height="${body_height}" />
-   </link>
+    <xacro:inertial_cylinder mass="2" radius="${body_diameter/2}" height="${body_height}" />
+  </link>
   <joint name="dummy_base_joint" type="fixed">
     <axis rpy="0 0 0" xyz="0 0 1"/>
     <parent link="main_body"/>
     <child link="dummy_link"/>
-    <origin xyz="0 0 0" />
+    <origin xyz="0 0 -0.02" />
   </joint>
-  <xacro:macro name="front_sensor_sup_link" params="name side y_pos">
+  <xacro:macro name="front_sensor_link" params="name side y_pos">
     <link name="${name}_front_sensor">
       <visual>
         <geometry>
-          <box size="0.05 0.05 0.05"/>
-        </geometry>
-        <origin xyz="0 0 -0.05"/>
+          <box size="0.02 0.02 0.02"/>
+        </geometry>
+        <origin xyz="-0.02 0 0" rpy="0 0 0"/>
         <material name="white"/>
       </visual>
       <collision>
         <geometry>
-          <box size="0.05 0.05 0.05"/>
-        </geometry>
-        <origin xyz="0 0 -0.05"/>
+          <box size="0.02 0.02 0.02"/>
+        </geometry>
+        <origin xyz="-0.02 0 0" rpy="0 0 0"/>
       </collision>
     </link>
     <joint name="${side}_front_base_joint" type="fixed">
-      <axis rpy="0 0 0" xyz="0 0 1"/>
+      <axis rpy="0 0 0" xyz="0 0 0"/>
       <parent link="main_body"/>
       <child link="${name}_front_sensor"/>
-      <origin xyz="${body_lenght/2} ${side*y_pos} 0.125" />
+      <origin xyz="${body_diameter/2} ${side*y_pos} 0" rpy="0 -0.15 0" />
     </joint>
     <gazebo reference="${name}_front_sensor">
@@ -97,7 +113,7 @@
          </scan>
          <range>
-            <min>0.01</min>
+            <min>0.05</min>
             <max>2</max>
-            <resolution>0.02</resolution>
+            <resolution>0.01</resolution>
          </range>
       </ray>
@@ -123,5 +139,5 @@
     </collision>
     <visual>
-      <origin xyz="0 0 0" rpy="0 0 0"/>
+      <origin xyz="0 0 ${-camera_link}" rpy="0 0 0"/>
       <geometry>
     <box size="${camera_link} ${camera_link} ${camera_link}"/>
@@ -130,5 +146,5 @@
     </visual>
     <inertial>
-      <mass value="1e-5" />
+      <mass value="1e-5"/>
       <origin xyz="0 0 0" rpy="0 0 0"/>
       <inertia ixx="1e-6" ixy="0" ixz="0" iyy="1e-6" iyz="0" izz="1e-6" />
@@ -137,5 +153,5 @@
   <joint name="camera_joint" type="fixed">
     <axis xyz="0 1 0" />
-    <origin xyz="${body_lenght/2} 0 0.125" rpy="0 0 0"/>
+    <origin xyz="${body_diameter/2} 0 ${body_height/2}" rpy="0 -0.15 0"/>
     <parent link="main_body"/>
     <child link="camera_link"/>
@@ -209,72 +225,38 @@
     <link name="${side}_aux_wheel">
       <visual>
-        <!-- origin xyz="0 ${reflect*aux_wheel_width/2} 0" rpy="${pi/2} 0 0" / -->
         <origin xyz="0 0 0" rpy="${pi/2} 0 0" />
         <geometry>
-          <cylinder radius="${aux_wheel_radius}" length="${aux_wheel_width}"/>
+          <sphere radius="${aux_wheel_radius}"/>
         </geometry>
         <material name="black"/>
       </visual>
       <collision>
-        <!-- origin xyz="0 ${reflect*aux_wheel_width/2} 0" rpy="${pi/2} 0 0" / -->
         <origin xyz="0 0 0" rpy="${pi/2} 0 0" />
         <geometry>
-          <cylinder radius="${aux_wheel_radius}" length="${aux_wheel_width}"/>
+          <sphere radius="${aux_wheel_radius}"/>
         </geometry>
       </collision>
       <!-- inertial>
-        <mass value="0.2" />
-        <inertia ixx="0.0001" ixy="0.0" ixz="0.0" iyy="0.00016" iyz="0.0" izz="0.0001" />
+        <mass value="0.05" />
+        <inertia ixx="0.0002" ixy="0.0" ixz="0.0" iyy="0.0002" iyz="0.0" izz="0.0002" />
       </inertial -->
-      <xacro:inertial_cylinder_y_axis mass="0.2" radius="${aux_wheel_radius}" height="${aux_wheel_width}" />
+      <xacro:inertial_sphere mass="0.05" radius="${aux_wheel_radius}" />
     </link>
     <joint name="${side}_aux_wheel_joint" type="continuous">
+      <parent link="main_body"/>
+      <child link="${side}_aux_wheel"/>
       <axis xyz="0 1 0" rpy="0 0 0" />
-      <parent link="${side}_front_support"/>
-      <child link="${side}_aux_wheel"/>
-      <origin xyz="-0.05 ${reflect*0.01} -0.07" rpy="0 0 0"/>
-      <!-- origin xyz="-0.03 0 -0.06" rpy="0 0 0"/ -->
+      <!-- origin xyz="${-body_diameter/2+0.05} ${reflect*0.01} -0.05" rpy="0 0 0"/ -->
+      <origin xyz="-0.12 ${reflect*0.01} -0.05" rpy="0 0 0"/>
     </joint>
     <!-- This block provides the simulator (Gazebo) with information on a few additional
     physical properties. See http://gazebosim.org/tutorials/?tut=ros_urdf for more-->
     <gazebo reference="${side}_aux_wheel">
-      <mu1 value="100.0"/>
-      <mu2 value="50.0"/>
-      <kp value="10000000.0" />
-      <kd value="1.0" />
+      <mu1 value="1.0"/>
+      <mu2 value="1.0"/>
+      <kp value="1000000.0" />
+      <kd value="100.0" />
       <material>Gazebo/Grey</material>
     </gazebo>
-  </xacro:macro>
-  <xacro:macro name="support" params="side displacement reflect">
-    <link name="${side}_front_support">
-      <visual>
-        <geometry>
-          <box size="0.05 0.01 0.08"/>
-        </geometry>
-        <!-- origin xyz="0 ${displacement} -0.04"/ -->
-        <origin xyz="-0.02 ${displacement} -0.04"/>
-        <material name="white"/>
-      </visual>
-      <collision>
-        <geometry>
-          <box size="0.05 0.01 0.08"/>
-        </geometry>
-        <!-- origin xyz="0 ${displacement} -0.04"/ -->
-        <origin xyz="-0.02 ${displacement} -0.04"/>
-      </collision>
-      <!-- inertial>
-        <mass value="0.2" />
-        <inertia ixx="0.0001" ixy="0.0" ixz="0.0" iyy="0.00016" iyz="0.0" izz="0.0001" />
-      </inertial -->
-      <xacro:inertial_cuboid mass="0.2" len="0.05" width="0.01" height="0.08" />
-    </link>
-    <joint name="${side}_front_base_joint" type="continuous">
-      <axis rpy="0 0 0" xyz="0 0 1"/>
-      <parent link="main_body"/>
-      <child link="${side}_front_support"/>
-      <origin xyz="0.3 ${reflect*0.15} -0.125" />
-      <dynamics damping="1" friction="0.1"/>
-    </joint>
-    <xacro:aux_wheel side="${side}"  reflect="${reflect}"/>
   </xacro:macro>
   <xacro:macro name="traction_wheel" params="side reflect">
@@ -293,15 +275,15 @@
         </geometry>
       </collision>
-      <!-- inertial>
-        <mass value="1" />
-        <inertia ixx="0.003" ixy="0.0" ixz="0.0" iyy="0.006" iyz="0.0" izz="0.003" />
-      </inertial -->
-      <xacro:inertial_cylinder_y_axis mass="1" radius="${traction_wheel_radius}" height="${traction_wheel_width}" />
-    </link>
+     <!-- inertial>
+      <mass value="0.1" />
+      <inertia ixx="0.00001" ixy="0.0" ixz="0.0" iyy="0.00009" iyz="0.0" izz="0.00001" />
+    </inertial -->
+    <xacro:inertial_cylinder_y_axis mass="0.1" radius="${traction_wheel_radius}" height="${traction_wheel_width}" />
+   </link>
     <joint name="${side}_traction_wheel_joint" type="continuous">
       <axis xyz="0 1 0" rpy="0 0 0" />
       <parent link="main_body"/>
       <child link="${side}_traction_wheel"/>
-      <origin xyz="-${body_lenght/3} ${reflect*(body_width/2+0.01)} ${-body_height/2}" rpy="0 0 0"/>
+      <origin xyz="${body_diameter/3} ${reflect*(body_diameter/3)} ${-body_height/2}" rpy="0 0 0"/>
     </joint>
     <!-- This block provides the simulator (Gazebo) with information on a few additional
@@ -311,6 +293,6 @@
       <mu2 value="100.0"/>
       <kp value="10000000.0" />
-      <kd value="1.0" />
-      <material>Gazebo/Grey</material>
+      <kd value="100.0" />
+      <material>Gazebo/Black</material>
     </gazebo>
     <!-- This block connects the wheel joint to an actuator (motor), which informs both
@@ -328,8 +310,7 @@
   <xacro:traction_wheel side="left" reflect="-1"/>
   <xacro:traction_wheel side="right" reflect="1"/>
-  <xacro:support side="left" displacement="${traction_wheel_width/3}" reflect="-1" />
-  <xacro:support side="right" displacement="${-traction_wheel_width/3}" reflect="1" />
-  <xacro:front_sensor_sup_link name="ultra_1" side="-1" y_pos="0.1" />
-  <xacro:front_sensor_sup_link name="ultra_2" side="1" y_pos="0.1" />
+  <xacro:aux_wheel side="center" reflect="0"/>
+  <xacro:front_sensor_link name="ultra_1" side="-1" y_pos="0.1" />
+  <xacro:front_sensor_link name="ultra_2" side="1" y_pos="0.1" />
   <!-- Gazebo plugin for ROS Control -->
   <gazebo>
